File: videoOSD.kicad_pcb (KiCad board)
At the start: 2 copper layers, 12 x 29 mm, 24 parts, among them U1 MAX7456EUI+, Y1 Crystal_GND24

Commit message: update
Parts:
- moved C3 0.25 mm to (134.2, 91.5)
Routing:
- net GND: track 10.9 -> 11.8 mm, vias 6 -> 7
Other:
- board text added: "Nic DeBruin 2026 Analog FPV OSD KV0R for WPI HPRC"
Changed lines of the file:
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@@
 			(at 1.23 0 90)
 			(layer "F.SilkS")
+			(hide yes)
 			(effects
 				(font
@@
 			(at 1.27 -0.5 90)
 			(layer "F.SilkS")
+			(hide yes)
 			(effects
 				(font
@@
 	(footprint "Capacitor_SMD:C_0402_1005Metric"
 		(layer "F.Cu")
-		(at 134.5 91.52 90)
+		(at 134.25 91.48 90)
 		(descr "Capacitor SMD 0402 (1005 Metric), square (rectangular) end terminal, IPC-7351 nominal, (Body size source: IPC-SM-782 page 76, https://www.pcb-3d.com/wordpress/wp-content/uploads/ipc-sm-782a_amendment_1_and_2.pdf), generated with kicad-footprint-generator")
 		(tags "capacitor")
 		(property "Reference" "C3"
-			(at -1.73 0 90)
+			(at -1.77 0.25 90)
 			(layer "F.SilkS")
 			(effects
@@
 		(layer "Edge.Cuts")
 	)
+	(gr_text "Nic DeBruin 2026\nAnalog FPV OSD\nKV0R for WPI HPRC"
+		(at 134.5 103 0)
+		(layer "F.Cu")
+		(effects
+			(font
+				(size 0.5 0.5)
+				(thickness 0.1)
+				(bold yes)
+			)
+			(justify right bottom)
+		)
+	)
 	(gr_text "OUT"
-		(at 125.2 95.5 270)
+		(at 125.25 95.5 270)
 		(layer "F.SilkS")
 		(effects
@@
 	)
 	(segment
-		(start 132.785 91.04)
-		(end 132.725 91.1)
-		(width 0.2)
-		(layer "F.Cu")
-		(net 1)
-	)
-	(segment
 		(start 128.7 89.8)
 		(end 127 89.8)
@@
 	)
 	(segment
+		(start 134.45 90)
+		(end 134.45 90.8)
+		(width 0.2)
+		(layer "F.Cu")
+		(net 1)
+	)
+	(segment
+		(start 132.825 91)
+		(end 132.725 91.1)
+		(width 0.2)
+		(layer "F.Cu")
+		(net 1)
+	)
+	(segment
+		(start 134.45 90.8)
+		(end 134.25 91)
+		(width 0.2)
+		(layer "F.Cu")
+		(net 1)
+	)
+	(segment
 		(start 133.1 97.85)
 		(end 133.35 97.85)
@@
 	)
 	(segment
+		(start 134.25 91)
+		(end 132.825 91)
+		(width 0.2)
+		(layer "F.Cu")
+		(net 1)
+	)
+	(segment
 		(start 127 87.85)
 		(end 126.06 87.85)
@@
 		(start 128.799265 89.700735)
 		(end 128.7 89.8)
-		(width 0.2)
-		(layer "F.Cu")
-		(net 1)
-	)
-	(segment
-		(start 134.5 91.04)
-		(end 132.785 91.04)
 		(width 0.2)
 		(layer "F.Cu")
@@
 	)
 	(via
+		(at 130 99.5)
+		(size 0.6)
+		(drill 0.3)
+		(layers "F.Cu" "B.Cu")
+		(free yes)
+		(net 1)
+	)
+	(via
 		(at 128.799265 89.5)
 		(size 0.6)
@@
 	)
 	(segment
-		(start 134.5 92)
-		(end 134.25 91.75)
-		(width 0.2)
-		(layer "F.Cu")
-		(net 2)
-	)
-	(segment
 		(start 131.5 91.75)
 		(end 132.725 91.75)
@@
 	)
 	(segment
-		(start 134.25 91.75)
-		(end 132.725 91.75)
-		(width 0.2)
-		(layer "F.Cu")
-		(net 2)
-	)
-	(segment
 		(start 125.46 91.46)
 		(end 125.5 91.5)
@@
 	)
 	(segment
+		(start 134.04 91.75)
+		(end 132.725 91.75)
+		(width 0.2)
+		(layer "F.Cu")
+		(net 2)
+	)
+	(segment
 		(start 127 90.45)
 		(end 129.2 90.45)
@@
 		(width 0.2)
 		(layer "F.Cu")
+		(net 2)
+	)
+	(segment
+		(start 134.25 91.96)
+		(end 134.04 91.75)
+		(width 0.2)
+		(layer "F.Cu")
