File: pcb/videoOSD.kicad_pcb (KiCad board)
At the start: 2 copper layers, 12 x 29 mm, 24 parts, among them U1 MAX7456EUI+, Y1 Crystal_GND24

Commit message: pcb done
Routing:
- net Net-(U1-XFB): track 10.0 -> 10.8 mm
Other:
- board text added: "Let's Build A Radio!"
